Commit message: Added L515 mesh

File: mcap/generalized_humanoid/GR1_model/GR1T2/urdf/GR1T2_simple_mod.urdf (robot description, URDF)
Before this commit: robot GR1T2Simple, 37 links, 36 joints
Links:
- link l515: geometry visual mesh filename=file:///home/jose/ws/ros2/foxglove_ws/src/foxglove_tutorial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
Joints:
- joint l515_j: origin xyz=0.0 0.0 0.0 rpy=-1.5707 0.0 -1.5707 -> xyz=0.115 0.0 0.2 rpy=-2.3561 0.0 -1.5707
