Commit message: Updated URDF paths

File: mcap/generalized_humanoid/GR1_model/GR1T2/GR1T2_simple_mod.urdf (robot description, URDF)
Before this commit: robot GR1T2, 35 links, 34 joints
Links:
- removed link link_head_pitch
- removed link link_head_roll
- removed link link_head_yaw
- removed link link_imu
- removed link link_torso
- removed link link_waist_pitch
- removed link link_waist_roll
- removed link link_waist_yaw
- added link base_link
- added link head_pitch, mass 0.00543512; visual mesh filename=meshes/head3.STL
- added link head_roll, mass 0.07131711; visual mesh filename=meshes/head2.STL
- added link head_yaw, mass 1.3898352; visual mesh filename=meshes/head1.STL
- added link l515; visual mesh filename=file:///home/jose/ws/ros2/foxglove_ws/src/foxglove_tutorial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
- added link torso
- added link waist_pitch, mass 2.90421452; visual mesh filename=meshes/waist2.STL
- added link waist_roll, mass 7.54469333; collision cylinder length=0.2 radius=0.1; visual mesh filename=meshes/waist1.STL
- added link waist_yaw, mass 0.50743792; visual mesh filename=meshes/waist3.STL
- added link z_link_imu; visual box size=0.05 0.05 0.02
- link base: geometry visual mesh filename=meshes/base.STL
- link l_foot_pitch: geometry visual mesh filename=meshes/Lleg5.STL
- link l_foot_roll: geometry collision cylinder length=0.24 radius=0.02; collision cylinder length=0.24 radius=0.02
- link l_hand_pitch: geometry collision sphere radius=0.036; visual mesh filename=meshes/Larm7.STL
- link l_hand_roll: geometry visual mesh filename=meshes/Larm6.STL
- link l_hand_yaw: geometry collision cylinder length=0.17 radius=0.035; visual mesh filename=meshes/Larm5.STL
- link l_lower_arm_pitch: geometry visual mesh filename=meshes/Larm4.STL
- link l_shank_pitch: geometry collision cylinder length=0.2 radius=0.05; visual mesh filename=meshes/Lleg4.STL
- link l_thigh_pitch: geometry collision cylinder length=0.35 radius=0.05; visual mesh filename=meshes/Lleg3.STL
- link l_thigh_roll: geometry visual mesh filename=meshes/Lleg1.STL
- link l_thigh_yaw: geometry visual mesh filename=meshes/Lleg2.STL
- link l_upper_arm_pitch: geometry visual mesh filename=meshes/Larm1.STL
- link l_upper_arm_roll: geometry visual mesh filename=meshes/Larm2.STL
- link l_upper_arm_yaw: geometry collision cylinder length=0.11 radius=0.03; visual mesh filename=meshes/Larm3.STL
- link r_foot_pitch: geometry visual mesh filename=meshes/Rleg5.STL
- link r_foot_roll: geometry collision cylinder length=0.24 radius=0.02; collision cylinder length=0.24 radius=0.02
- link r_hand_pitch: geometry collision sphere radius=0.036; visual mesh filename=meshes/Rarm7.STL
- link r_hand_roll: geometry visual mesh filename=meshes/Rarm6.STL
- link r_hand_yaw: geometry collision cylinder length=0.17 radius=0.035; visual mesh filename=meshes/Rarm5.STL
- link r_lower_arm_pitch: geometry visual mesh filename=meshes/Rarm4.STL
- link r_shank_pitch: geometry collision cylinder length=0.2 radius=0.05; visual mesh filename=meshes/Rleg4.STL
- link r_thigh_pitch: geometry collision cylinder length=0.35 radius=0.05; visual mesh filename=meshes/Rleg3.STL
- link r_thigh_roll: geometry visual mesh filename=meshes/Rleg1.STL
- link r_thigh_yaw: geometry visual mesh filename=meshes/Rleg2.STL
- link r_upper_arm_pitch: geometry visual mesh filename=meshes/Rarm1.STL
- link r_upper_arm_roll: geometry visual mesh filename=meshes/Rarm2.STL
- link r_upper_arm_yaw: geometry collision cylinder length=0.11 radius=0.03; visual mesh filename=meshes/Rarm3.STL
Joints:
- removed joint joint_imu
- removed joint joint_waist_pitch
- removed joint joint_waist_roll
- removed joint joint_waist_yaw
- added joint base_j: type fixed, parent base_link, child base
- added joint l515_j: type fixed, parent head_yaw, child l515, origin xyz=0.115 0.0 0.2 rpy=-2.3561 0.0 -1.5707
- added joint waist_pitch: type revolute, parent waist_yaw, child waist_pitch, origin xyz=0 0 0.0570000000000001 rpy=0 0 0, axis 0 1 0, limit lower=-0.52 upper=1.22 effort=66 velocity=16.76
- added joint waist_roll: type revolute, parent waist_pitch, child waist_roll, origin xyz=0 0 0.081 rpy=0 0 0, axis 1 0 0, limit lower=-0.7 upper=0.7 effort=66 velocity=16.76
- added joint waist_yaw: type revolute, parent base, child waist_yaw, origin xyz=0 0 0.00649999999999984 rpy=0 0 0, axis 0 0 1, limit lower=-1.05 upper=1.05 effort=66 velocity=16.76
- added joint z_joint_imu: type fixed, parent base, child z_link_imu, origin xyz=-0.0645 0 -0.102 rpy=0 0 0
- joint joint_head_pitch: child link_head_pitch -> head_pitch; parent link_torso -> torso
- joint joint_head_roll: child link_head_roll -> head_roll; parent link_head_pitch -> head_pitch
- joint joint_head_yaw: child link_head_yaw -> head_yaw; parent link_head_roll -> head_roll
- joint joint_torso: child link_torso -> torso; parent link_waist_roll -> waist_roll
- joint l_elbow_pitch: origin xyz=0 0.00125501157055688 -0.188749174791823 rpy=0 0 0 -> xyz=0 0.00125501157055688 -0.188749174791823 rpy=0 -0.3 0
- joint l_shoulder_pitch: parent link_torso -> torso
- joint l_shoulder_roll: origin xyz=0 0.0669999999997965 0 rpy=-0.436334785573203 0 0 -> xyz=0 0.067 0 rpy=-0.2364 0 0
- joint r_elbow_pitch: origin xyz=0 0 -0.188530330300762 rpy=0 0 0 -> xyz=0 0 -0.188530330300762 rpy=0 -0.3 0
- joint r_shoulder_pitch: parent link_torso -> torso
- joint r_shoulder_roll: origin xyz=0 -0.0670000000000026 0 rpy=0.436332306093773 0 0 -> xyz=0 -0.067 0 rpy=0.23627 0 0
