Commit message: Fix depth camera, robot position and box image and position

File: integrations/ros2/gazebo/urdf/foxglove_box.urdf (robot description, URDF)
Before this commit: robot foxglove_block, 1 links, 0 joints
Links:
- link root_link: geometry collision box size=0.04 0.1705 0.04; visual mesh filename=package://fg_gazebo_example/meshes/foxglove_box.dae scale=0.02 0.02 0.02

File: integrations/ros2/gazebo/urdf/robot.xacro (robot description, xacro)
@@ -13,5 +13,8 @@
        those URDFs has this "world"-named-root-link quirk and their spawn args are
        honored normally. -->
-  <xacro:property name="arm_x" value="1.0" />
+  <!-- arm_x: table is 1.0m long in X (see arm_table_top in foxglove_demo.sdf);
+       sit 0.25 table-lengths back from center so the wrist camera has a clearer
+       look at the Foxglove box toward +X. -->
+  <xacro:property name="arm_x" value="0.75" />
   <xacro:property name="arm_y" value="-3.5" />
   <!-- arm_z = table_height: the arm sits on top of the table at this position (see
@@ -29,5 +32,5 @@
     <parent link="world" />
     <child link="podest" />
-    <origin xyz="${arm_x} ${arm_y} ${arm_z}" rpy="0 0 0" />
+    <origin xyz="${arm_x} ${arm_y} ${arm_z + podest_height/2}" rpy="0 0 0" />
   </joint>
   <!-- Small podest so the arm isn't floating at the origin -->
